File: CH340E-UnoC_DRV8830/CH340E-UnoC_DRV8830.kicad_sch (KiCad schematic)
At the start: 87 parts, among them J1 Power, J3 Analog, J4 Digital/PWM

Commit message: feat: Schematic PDFs added.
Parts:
- removed JP?: A0IC1-DNP, symbol Jumper:SolderJumper_2_Open
- added F?: MF-MSMF150_24X-2/1.5A, FUSC4632X160N, symbol Fuse_MF-MSMF150_24X-2_1812 (4532 Metric)_SamacSys:MF-MSMF150_24X-2
- added JP?: A0IC1-DNP, symbol Jumper:SolderJumper_2_Bridged
Connections:
- net +5V: now also F?.1; no longer D?.2
- net A0_IC1: now also JP?.1 (A)
- net DRV_VCC: now also JP?.2 (B)
- new net: D?.2, F?.2
Other:
- note added: "4.5V~21V"
- note added: "オープンではなく、GND接置してあるため注意 IC1 A0=1, A1=0 IC2 A0=0, A1=0"
- moved on the sheet: C?, D?, JP?, L?
